File: Home assistant/Xmas tree/PCB/Xmas tree.brd (EAGLE design)
At the start: 64 x 38 mm, 12 parts, among them T1 BC547, X1 3PIN_5MM_TERMINAL

Commit message: Xmas tree update
Parts:
- R1: value 10k -> 470R
- moved R1 0.86 mm to (34.0, 19.7)
Connections:
- net N$1 renamed +12VAC
- net N$2 renamed -12VAC
- net N$3 renamed 12VDC
- net N$6: now also U$1.JP2.4; no longer U$1.JP2.6
Routing:
- net N$6: track 6.42 -> 3.53 mm
- net N$4: track 9.42 -> 9.98 mm
Changed lines of the file:
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@@
 <setting verticaltext="up"/>
 </settings>
-<grid distance="0.5" unitdist="mm" unit="mm" style="lines" multiple="1" display="no" altdistance="5" altunitdist="mil" altunit="mil"/>
+<grid distance="0.25" unitdist="mm" unit="mm" style="lines" multiple="1" display="no" altdistance="5" altunitdist="mil" altunit="mil"/>
 <layers>
 <layer number="1" name="Top" color="4" fill="1" visible="yes" active="yes"/>
@@
 <elements>
 <element name="C1" library="resistor" package="E3,5-10" package3d_urn="urn:adsk.eagle:package:23351/1" value="1000uF" x="33.925" y="29.21" smashed="yes" rot="R270">
-<attribute name="NAME" x="28.854" y="23.354" size="1.27" layer="25" ratio="10"/>
+<attribute name="NAME" x="28.604" y="23.354" size="1.27" layer="25" ratio="10"/>
 <attribute name="VALUE" x="30.877" y="32.512" size="1.27" layer="27" ratio="10" rot="R270"/>
 </element>
 <element name="D1" library="diode" library_urn="urn:adsk.eagle:library:210" package="DO41-10" package3d_urn="urn:adsk.eagle:package:43336/1" value="1N4004" x="10.52" y="25.025" smashed="yes" rot="R90">
-<attribute name="NAME" x="8.869" y="22.993" size="1.27" layer="25" ratio="10" rot="R90"/>
+<attribute name="NAME" x="8.869" y="24.993" size="1.27" layer="25" ratio="10" rot="R90"/>
 <attribute name="POPULARITY" value="82" x="10.52" y="25.025" size="1.778" layer="27" rot="R90" display="off"/>
 </element>
 <element name="D2" library="diode" library_urn="urn:adsk.eagle:library:210" package="DO41-10" package3d_urn="urn:adsk.eagle:package:43336/1" value="1N4004" x="10.52" y="12.055" smashed="yes" rot="R270">
-<attribute name="NAME" x="7.726" y="12.182" size="1.27" layer="25" ratio="10" rot="R270"/>
+<attribute name="NAME" x="7.476" y="13.932" size="1.27" layer="25" ratio="10" rot="R270"/>
 <attribute name="POPULARITY" value="82" x="10.52" y="12.055" size="1.778" layer="27" rot="R270" display="off"/>
 </element>
 <element name="D3" library="diode" library_urn="urn:adsk.eagle:library:210" package="DO41-10" package3d_urn="urn:adsk.eagle:package:43336/1" value="1N4004" x="16.87" y="25.025" smashed="yes" rot="R270">
-<attribute name="NAME" x="14.076" y="25.152" size="1.27" layer="25" ratio="10" rot="R270"/>
+<attribute name="NAME" x="14.076" y="27.152" size="1.27" layer="25" ratio="10" rot="R270"/>
 <attribute name="POPULARITY" value="82" x="16.87" y="25.025" size="1.778" layer="27" rot="R270" display="off"/>
 </element>
 <element name="D4" library="diode" library_urn="urn:adsk.eagle:library:210" package="DO41-10" package3d_urn="urn:adsk.eagle:package:43336/1" value="1N4004" x="16.87" y="12.055" smashed="yes" rot="R90">
-<attribute name="NAME" x="15.219" y="10.023" size="1.27" layer="25" ratio="10" rot="R90"/>
+<attribute name="NAME" x="15.219" y="11.773" size="1.27" layer="25" ratio="10" rot="R90"/>
 <attribute name="POPULARITY" value="82" x="16.87" y="12.055" size="1.778" layer="27" rot="R90" display="off"/>
 </element>
@@
 <attribute name="NAME" x="42.855" y="18.915" size="1.27" layer="21"/>
 </element>
-<element name="R1" library="resistor" package="0207/10" package3d_urn="urn:adsk.eagle:package:23491/1" value="10k" x="34" y="18.845" smashed="yes">
-<attribute name="NAME" x="30.952" y="20.369" size="1.27" layer="25" ratio="10"/>
-<attribute name="VALUE" x="31.7394" y="18.21" size="1.27" layer="27" ratio="10"/>
+<element name="R1" library="resistor" package="0207/10" package3d_urn="urn:adsk.eagle:package:23491/1" value="470R" x="34" y="19.7" smashed="yes">
+<attribute name="NAME" x="29.952" y="16.724" size="1.27" layer="25" ratio="10"/>
+<attribute name="VALUE" x="33.9894" y="16.815" size="1.27" layer="27" ratio="10"/>
 </element>
 <element name="SD1" library="Voltage" package="TRACO_TSR_1-2450" value="TRACO_TSR_1-2450" x="45.355" y="28.575" smashed="yes" rot="R270">
@@
 <element name="T1" library="transistor" library_urn="urn:adsk.eagle:library:402" package="TO92-CBE" package3d_urn="urn:adsk.eagle:package:29921/2" value="BC547" x="34.065" y="12.075" smashed="yes" rot="R180">
 <attribute name="NAME" x="30.89" y="11.44" size="1.27" layer="25" ratio="10" rot="R180"/>
+<attribute name="POPULARITY" value="0" x="34.065" y="12.075" size="1.778" layer="27" rot="R180" display="off"/>
 </element>
 <element name="U$1" library="Sbirka modulu" package="WEMOS-D1-MINI" value="WEMOS-D1-MINI" x="13.97" y="17.78" smashed="yes"/>
 <element name="X1" library="Terminaly" package="3PIN_5MM_TERMINAL" value="3PIN_5MM_TERMINAL" x="56.025" y="28.065" smashed="yes" rot="R270">
-<attribute name="NAME" x="61.8019" y="22.067" size="1.27" layer="25" rot="R270"/>
+<attribute name="NAME" x="50.5519" y="22.067" size="1.27" layer="25" rot="R270"/>
 </element>
 </elements>
@@
 <contactref element="U$1" pad="JP1.8"/>
 </signal>
-<signal name="N$1">
+<signal name="+12VAC">
 <contactref element="D1" pad="A"/>
 <contactref element="D3" pad="C"/>
@@
 <wire x1="22.5" y1="33.5" x2="50.59" y2="33.5" width="1.27" layer="16"/>
 </signal>
-<signal name="N$2">
+<signal name="-12VAC">
 <contactref element="D2" pad="A"/>
 <contactref element="D4" pad="C"/>
@@
 <wire x1="53.395" y1="35.695" x2="12.2" y2="35.695" width="1.27" layer="16"/>
 </signal>
-<signal name="N$3">
+<signal name="12VDC">
 <contactref element="D1" pad="C"/>
 <contactref element="D2" pad="C"/>
@@
 <wire x1="43.605" y1="31.125" x2="34.062" y2="31.125" width="1.27" layer="16"/>
 <wire x1="33.925" y1="30.988" x2="34.062" y2="31.125" width="1.27" layer="16"/>
-<wire x1="33.925" y1="30.988" x2="23.468" y2="30.988" width="1.27" layer="16"/>
-<wire x1="23.468" y1="30.988" x2="12.425" y2="19.945" width="1.27" layer="16"/>
-<wire x1="12.425" y1="19.945" x2="10.52" y2="19.945" width="1.27" layer="16"/>
+<wire x1="23.468" y1="30.988" x2="33.925" y2="30.988" width="1.27" layer="16"/>
+<wire x1="10.52" y1="19.945" x2="12.425" y2="19.945" width="1.27" layer="16"/>
+<wire x1="12.425" y1="19.945" x2="23.468" y2="30.988" width="1.27" layer="16"/>
 </signal>
 <signal name="GND">
@@
 <contactref element="T1" pad="B"/>
 <contactref element="R1" pad="2"/>
-<wire x1="39.08" y1="18.845" x2="38.082971875" y2="18.845" width="1.27" layer="16"/>
-<wire x1="38.082971875" y1="18.845" x2="34.065" y2="14.802990625" width="1.27" layer="16"/>
+<wire x1="39.08" y1="19.7" x2="39.077021875" y2="19.845" width="1.27" layer="16"/>
+<wire x1="39.077021875" y1="19.845" x2="34.065" y2="14.802990625" width="1.27" layer="16"/>
 <wire x1="34.065" y1="14.802990625" x2="34.065" y2="12.075" width="1.27" layer="16"/>
 </signal>
 <signal name="N$6">
-<contactref element="U$1" pad="JP2.6"/>
 <contactref element="R1" pad="1"/>
-<wire x1="25.4" y1="14.605" x2="26.605" y2="14.605" width="1.27" layer="16"/>
-<wire x1="28.95" y1="16.95" x2="28.92" y2="18.845" width="1.27" layer="16"/>
-<wire x1="26.605" y1="14.605" x2="28.95" y2="16.95" width="1.27" layer="16"/>
+<contactref element="U$1" pad="JP2.4"/>
+<wire x1="25.5" y1="19.685" x2="25.4" y2="19.685" width="0.1524" layer="16"/>
+<wire x1="28.92" y1="19.7" x2="25.515" y2="19.7" width="1.27" layer="16"/>
+<wire x1="25.515" y1="19.7" x2="25.5" y2="19.685" width="0.1524" layer="16"/>
 </signal>
 <signal name="N$5">
