File: Home assistant/Xmas tree/PCB/Xmas tree.sch (EAGLE design)
At the start: 12 parts, among them T1 BC547, X1 3PIN_5MM_TERMINAL

Commit message: Xmas tree update
Parts:
- R1: value 10k -> 470R
Connections:
- net N$1 renamed +12VAC
- net N$2 renamed -12VAC
- net N$3 renamed 12VDC
- net N$6: now also U$1.D2; no longer U$1.D4
Changed lines of the file:
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@@
 <?xml version="1.0" encoding="utf-8"?>
 <!DOCTYPE eagle SYSTEM "eagle.dtd">
-<eagle version="9.2.2">
+<eagle version="9.6.2">
 <drawing>
 <settings>
@@
 <part name="C1" library="resistor" deviceset="CPOL-EU" device="E3.5-10" package3d_urn="urn:adsk.eagle:package:23351/1" value="1000uF"/>
 <part name="SD1" library="Voltage" deviceset="TRACO_TSR_1-2450" device=""/>
-<part name="GND1" library="supply1" deviceset="GND" device=""/>
-<part name="P+1" library="supply1" deviceset="+5V" device=""/>
+<part name="GND1" library="supply1" library_urn="urn:adsk.eagle:library:371" deviceset="GND" device=""/>
+<part name="P+1" library="supply1" library_urn="urn:adsk.eagle:library:371" deviceset="+5V" device=""/>
 <part name="U$1" library="Sbirka modulu" deviceset="WEMOS-D1-MINI" device=""/>
-<part name="GND2" library="supply1" deviceset="GND" device=""/>
-<part name="P+2" library="supply1" deviceset="+5V" device=""/>
+<part name="GND2" library="supply1" library_urn="urn:adsk.eagle:library:371" deviceset="GND" device=""/>
+<part name="P+2" library="supply1" library_urn="urn:adsk.eagle:library:371" deviceset="+5V" device=""/>
 <part name="RL1" library="Rele_Finder" deviceset="36.11" device=""/>
 <part name="D5" library="diode" library_urn="urn:adsk.eagle:library:210" deviceset="1N4004" device="" package3d_urn="urn:adsk.eagle:package:43336/1"/>
 <part name="T1" library="transistor" library_urn="urn:adsk.eagle:library:402" deviceset="*-NPN-" device="TO92-CBE" package3d_urn="urn:adsk.eagle:package:29921/2" technology="BC547" value="BC547"/>
-<part name="R1" library="resistor" deviceset="R-EU_" device="0207/10" package3d_urn="urn:adsk.eagle:package:23491/1" value="10k"/>
-<part name="GND4" library="supply1" deviceset="GND" device=""/>
-<part name="P+4" library="supply1" deviceset="+5V" device=""/>
+<part name="R1" library="resistor" deviceset="R-EU_" device="0207/10" package3d_urn="urn:adsk.eagle:package:23491/1" value="470R"/>
+<part name="GND4" library="supply1" library_urn="urn:adsk.eagle:library:371" deviceset="GND" device=""/>
+<part name="P+4" library="supply1" library_urn="urn:adsk.eagle:library:371" deviceset="+5V" device=""/>
 </parts>
 <sheets>
@@
 </busses>
 <nets>
-<net name="N$1" class="0">
+<net name="+12VAC" class="0">
 <segment>
 <pinref part="D1" gate="1" pin="A"/>
@@
 </segment>
 </net>
-<net name="N$2" class="0">
+<net name="-12VAC" class="0">
 <segment>
 <pinref part="D2" gate="1" pin="A"/>
@@
 </segment>
 </net>
-<net name="N$3" class="0">
+<net name="12VDC" class="0">
 <segment>
 <pinref part="D1" gate="1" pin="C"/>
@@
 <net name="N$6" class="0">
 <segment>
-<pinref part="U$1" gate="G$1" pin="D4"/>
-<wire x1="129.54" y1="73.66" x2="137.16" y2="73.66" width="0.1524" layer="91"/>
-<wire x1="137.16" y1="73.66" x2="137.16" y2="119.38" width="0.1524" layer="91"/>
 <pinref part="R1" gate="G$1" pin="1"/>
+<wire x1="137.16" y1="78.74" x2="137.16" y2="119.38" width="0.1524" layer="91"/>
 <wire x1="137.16" y1="119.38" x2="101.6" y2="119.38" width="0.1524" layer="91"/>
-</segment>
-</net>
+<pinref part="U$1" gate="G$1" pin="D2"/>
+<wire x1="129.54" y1="78.74" x2="137.16" y2="78.74" width="0.1524" layer="91"/>
+</segment>
+</net>
