File: Citroen C5 X7/LED ambilight/PCB/C5 Ambilight.brd (EAGLE design)
At the start: 65 x 45 mm, 21 parts, among them Q1 SQP90P06-07L_GE3, X1 2PIN_5MM_TERMINAL, X2 2PIN_5MM_TERMINAL, X3 JST-XH-03-PIN-ROUND-PAD

Commit message: Updated PCB
Parts:
- R2: value 12k -> 10k
- R3: value 470R -> 10k
Changed lines of the file:
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@@
 <attribute name="VALUE" x="48.123" y="7.5438" size="1.27" layer="27" ratio="10" rot="R180"/>
 </element>
-<element name="R2" library="resistor" package="0207/7" package3d_urn="urn:adsk.eagle:package:23493/1" value="12k" x="23.055" y="40.962" smashed="yes" rot="R180">
+<element name="R2" library="resistor" package="0207/7" package3d_urn="urn:adsk.eagle:package:23493/1" value="10k" x="23.055" y="40.962" smashed="yes" rot="R180">
 <attribute name="NAME" x="21.785" y="39.565" size="1.27" layer="25" ratio="10" rot="R180"/>
 <attribute name="VALUE" x="26.738" y="39.6158" size="1.27" layer="27" ratio="10" rot="R180"/>
 </element>
-<element name="R3" library="resistor" package="0207/7" package3d_urn="urn:adsk.eagle:package:23493/1" value="470R" x="23.055" y="36.39" smashed="yes" rot="R180">
+<element name="R3" library="resistor" package="0207/7" package3d_urn="urn:adsk.eagle:package:23493/1" value="10k" x="23.055" y="36.39" smashed="yes" rot="R180">
 <attribute name="NAME" x="21.912" y="34.612" size="1.27" layer="25" ratio="10" rot="R180"/>
 <attribute name="VALUE" x="26.865" y="34.6628" size="1.27" layer="27" ratio="10" rot="R180"/>

Commit message: Fix capacitor value
Parts:
- C2, C3: value 1nF -> 1uF
Changed lines of the file:
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@@
 <attribute name="NAME" x="62.604" y="32.258" size="1.27" layer="25" rot="R90" align="top-left"/>
 </element>
-<element name="C2" library="resistor" package="C050-025X075" package3d_urn="urn:adsk.eagle:package:23637/1" value="1nF" x="38.481" y="26.67" smashed="yes" rot="R180">
+<element name="C2" library="resistor" package="C050-025X075" package3d_urn="urn:adsk.eagle:package:23637/1" value="1uF" x="38.481" y="26.67" smashed="yes" rot="R180">
 <attribute name="NAME" x="35.052" y="28.194" size="1.27" layer="25" ratio="10"/>
 <attribute name="VALUE" x="39.243" y="28.321" size="1.27" layer="27" ratio="10"/>
 </element>
-<element name="C3" library="resistor" package="C050-025X075" package3d_urn="urn:adsk.eagle:package:23637/1" value="1nF" x="6.477" y="23.368" smashed="yes">
+<element name="C3" library="resistor" package="C050-025X075" package3d_urn="urn:adsk.eagle:package:23637/1" value="1uF" x="6.477" y="23.368" smashed="yes">
 <attribute name="NAME" x="2.921" y="20.447" size="1.27" layer="25" ratio="10"/>
 <attribute name="VALUE" x="7.366" y="20.447" size="1.27" layer="27" ratio="10"/>
